File: Board1/TheHub.sch (KiCad schematic (older format))
At the start: 4 parts

Commit message: Add PCA9685, ADS1115, and hookups for different parts on i2c bus
Parts:
- added C? (x2): 10U, symbol C
- added J?: CONN_02X15, symbol CONN_02X15
- added J?: ARM_PWM_OUT, symbol CONN_01X16
- added J?: SCIENCE_PWM_OUT, symbol CONN_01X16
- added J?: WHEEL_PWM_OUT, symbol CONN_01X16
- added J?: ARM_ADC_1, symbol CONN_01X04
- added J?: ARM_ADC_2, symbol CONN_01X04
- added J?: SCI_ADC_1, symbol CONN_01X04
- added J?: WHEEL_ADC_1, symbol CONN_01X04
- added R? (x6): 2.2K, symbol R
- added U? (x4): PRE-ADS1115, symbol PRE-ADS1115
- added U? (x3): PRE-PCA9685, symbol PRE-PCA9685
- U?: Digikey (none) -> https://www.digikey.com/product-detail/en/stmicroelectronic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
Connections:
- net 3V3 is gone; now on net +3V3: J?.16 (P16)
- net +12V: now also C?.1
- net +3V3: now also C?.1, J?.3 (P3), R?.1, R?.1, R?.1, R?.1, R?.1, R?.1, U?.1 (VDD), U?.1 (VDD), U?.1 (VDD), U?.1 (VDD), U?.5 (ADDR), U?.5 (VCC), U?.5 (VCC), U?.5 (VCC)
- net 5V: now also J?.23 (P23)
- net GND: now also C?.2, C?.2, J?.24 (P24), J?.27 (P27), U?.1 (GND), U?.1 (GND), U?.1 (GND), U?.2 (GND), U?.2 (GND), U?.2 (GND), U?.2 (GND), U?.5 (ADDR)
- new net: J?.4 (P4), U?.10 (A3) (x4)
- new net: J?.1 (P1), U?.7 (A0) (x4)
- new net: J?.2 (P2), U?.8 (A1) (x4)
- new net: J?.3 (P3), U?.9 (A2) (x4)
- new net: J?.4 (P4), U?.10 (PWM3) (x3)
- new net: J?.5 (P5), U?.11 (PWM4) (x3)
- new net: J?.6 (P6), U?.12 (PWM5) (x3)
- new net: J?.7 (P7), U?.13 (PWM6) (x3)
- new net: J?.8 (P8), U?.14 (PWM7) (x3)
- new net: J?.9 (P9), U?.15 (PWM8) (x3)
- new net: J?.10 (P10), U?.16 (PWM9) (x3)
- new net: J?.11 (P11), U?.17 (PWM10) (x3)
- new net: J?.12 (P12), U?.18 (PWM11) (x3)
- new net: J?.13 (P13), U?.19 (PWM12) (x3)
- new net: J?.14 (P14), U?.20 (PWM13) (x3)
- new net: J?.15 (P15), U?.21 (PWM14) (x3)
- new net: J?.16 (P16), U?.22 (PWM15) (x3)
- new net: J?.1 (P1), U?.7 (PWM0) (x3)
- new net: J?.2 (P2), U?.8 (PWM1) (x3)
- new net: J?.3 (P3), U?.9 (PWM2) (x3)
- new net A0: J?.7 (P7)
- new net A1: J?.9 (P9)
- new net A2: J?.11 (P11)
- new net A3: J?.13 (P13)
- new net A4: J?.15 (P15), R?.2
- new net A5: J?.17 (P17), R?.2
- new net A6: J?.19 (P19)
- new net A7: J?.21 (P21)
- new net D10: J?.6 (P6)
- new net D11: J?.4 (P4)
- new net D12: J?.2 (P2)
- new net D13: J?.1 (P1)
- new net D2: J?.22 (P22)
- new net D3: J?.20 (P20)
- new net D4: J?.18 (P18)
- new net D5: J?.16 (P16)
- new net D6: J?.14 (P14)
- new net D7: J?.12 (P12)
- new net D8: J?.10 (P10)
- new net D9: J?.8 (P8)
- new net REF: J?.5 (P5)
- new net RST: J?.25 (P25), J?.26 (P26)
- new net RX0: J?.28 (P28)
- new net SCL_0: R?.2, U?.3 (SCL), U?.3 (SCL), U?.3 (SCL), U?.3 (SCL), U?.3 (SCL), U?.3 (SCL), U?.3 (SCL), U?.5 (ADDR)
- new net SCL_2: R?.2
- new net SDA_0: R?.2, U?.4 (SDA), U?.4 (SDA), U?.4 (SDA), U?.4 (SDA), U?.4 (SDA), U?.4 (SDA), U?.4 (SDA), U?.5 (ADDR)
- new net SDA_2: R?.2
- new net TX1: J?.30 (P30)
- new net VIN: J?.29 (P29)
- no-connect marks 9 -> 15
Other:
- note added: "0X48\n"
- note added: "0X49"
- note added: "0X4A"
- note added: "0X4B"
- note added: "ARM CARD"
- note added: "AUTONOMY CARD"
- note added: "SCIENCE CARD"
- note added: "SOLDER 00000: 0X40"
- note added: "SOLDER 00001: 0X41"
- note added: "SOLDER 00010: 0X42"
- note added: "WHEEL CARD"
