File: Board1/TheHub.sch (KiCad schematic (older format))
At the start: 54 parts, among them J1 ARM_ADC_1, J10 SCIENCE + WHEELS POWER CONN, J11 RFD900, J12 I2C_1 Test Point, J13 I2C_2 Test Point, J14 ARDUINO NANO LEFT, J15 GPIO Test, J16 I2C_3 Test Point, J17 12V OUT, J18 7.4V IN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

Commit message: Change 3v3 regulator, change appropriate pins to sockets
Parts:
- removed J5: NucleoF411RE, Pin_Headers:Pin_Header_Straight_2x19_Pitch2.54mm, symbol NucleoF411RE
- removed U6: LD1086DT33TR, symbol LD1086DT33TR
- added J23: NucleoRight, Socket_Strips:Socket_Strip_Straight_2x19_Pitch2.54mm, symbol CONN_02X19
- added J5: NucleoLeft, Socket_Strips:Socket_Strip_Straight_2x19_Pitch2.54mm, symbol CONN_02X19
- added U6: TL1963, TO_SOT_Packages_SMD:SOT-223-3Lead_TabPin2, symbol TL1963
- J11: footprint Pin_Headers:Pin_Header_Straight_2x08_Pitch2.54mm -> Socket_Strips:Socket_Strip_Angled_2x08_Pitch2.54mm
- J14, J22: footprint Pin_Headers:Pin_Header_Straight_1x15_Pitch2.54mm -> Socket_Strips:Socket_Strip_Straight_1x15_Pitch2.54mm
- J20: footprint Pin_Headers:Pin_Header_Straight_1x09_Pitch2.54mm -> Socket_Strips:Socket_Strip_Straight_1x09_Pitch2.54mm
- J21: footprint Pin_Headers:Pin_Header_Straight_1x06_Pitch2.54mm -> Socket_Strips:Socket_Strip_Straight_1x06_Pitch2.54mm
- R10, R11, R12, R13, R3, R4, R5: footprint (none) -> Resistors_SMD:R_0805
- U1, U4: footprint (none) -> FoxWestern:PCA9685
- U2, U3, U5, U9: footprint (none) -> Socket_Strips:Socket_Strip_Straight_1x10_Pitch2.54mm
- U7: footprint (none) -> TO_SOT_Packages_SMD:SOT-223-3Lead_TabPin2
Connections:
- net +12V: now also U6.1 (INPUT)
- net +3V3: now also J5.16 (P16), U6.3 (OUTPUT)
- net +5V: now also J5.18 (P18)
- net A4: now also J23.31 (P31)
- net A5: now also J23.25 (P25)
- net AGND: now also J23.32 (P32)
- net AVDD: now also J23.7 (P7)
- net BOOT0: now also J5.7 (P7)
- net E5V: now also J5.6 (P6)
- net GND: now also J23.20 (P20), J23.9 (P9), J5.19 (P19), J5.20 (P20), J5.22 (P22), J5.8 (P8), U6.2 (GND)
- net IOREF: now also J5.12 (P12)
- net PA0: now also J5.28 (P28)
- net PA1: now also J5.30 (P30)
- net PA10: now also J23.33 (P33)
- net PA11: now also J23.14 (P14)
- net PA12: now also J23.12 (P12)
- net PA13: now also J5.13 (P13)
- net PA14: now also J5.15 (P15)
- net PA15: now also J5.17 (P17)
- net PA2: now also J23.35 (P35)
- net PA3: now also J23.37 (P37)
- net PA4: now also J5.32 (P32)
- net PA5: now also J23.11 (P11)
- net PA6: now also J23.13 (P13)
- net PA7: now also J23.15 (P15)
- net PA8: now also J23.23 (P23)
- net PA9: now also J23.21 (P21)
- net PB0: now also J5.34 (P34)
- net PB1: now also J23.24 (P24)
- net PB12: now also J23.16 (P16)
- net PB13: now also J23.30 (P30)
- net PB14: now also J23.28 (P28)
- net PB15: now also J23.26 (P26)
- net PB2: now also J23.22 (P22)
- net PB4: now also J23.27 (P27)
- net PB5: now also J23.29 (P29)
- net PB6: now also J23.17 (P17)
- net PB7: now also J5.21 (P21)
- net PB8: now also J23.3 (P3)
- net PB9: now also J23.5 (P5)
- net PC0: now also J5.38 (P38)
- net PC1: now also J5.36 (P36)
- net PC10: now also J5.1 (P1)
- net PC11: now also J5.2 (P2)
- net PC12: now also J5.3 (P3)
- net PC13: now also J5.23 (P23)
- net PC14: now also J5.25 (P25)
- net PC15: now also J5.27 (P27)
- net PC2: now also J5.35 (P35)
- net PC3: now also J5.37 (P37)
- net PC4: now also J23.34 (P34)
- net PC5: now also J23.6 (P6)
- net PC6: now also J23.4 (P4)
- net PC7: now also J23.19 (P19)
- net PC8: now also J23.2 (P2)
- net PC9: now also J23.1 (P1)
- net PD2: now also J5.4 (P4)
- net PH0: now also J5.29 (P29)
- net PH1: now also J5.31 (P31)
- net RESET: now also J5.14 (P14)
- net U5V: now also J23.8 (P8)
- net VBAT: now also J5.33 (P33)
- net VDD: now also J5.5 (P5)
Changed lines of the file:
@@
 GND
-$Comp
-L LD1086DT33TR U6
-U 1 1 5935FC95
-P 9900 1650
-F 0 "U6" H 10250 1350 60  0000 C CNN
-F 1 "LD1086DT33TR" H 9850 1850 60  0000 C CNN
-F 2 "" H 9800 1700 60  0001 C CNN
-F 3 "" H 9800 1700 60  0001 C CNN
-F 4 "https://www.digikey.com/product-detail/en/stmicroelectronics/LD1086DT33TR/497-3446-1-ND/669240" H 9900 1650 60  0001 C CNN "Digikey"
-	1    9900 1650
-	1    0    0    -1
-$EndComp
 $Comp
 L +12V #PWR01
@@
 F 0 "U2" H 5450 5000 60  0000 C CNN
 F 1 "PRE-ADS1115" H 5250 6100 60  0000 C CNN
-F 2 "" H 5250 5750 60  0001 C CNN
+F 2 "Socket_Strips:Socket_Strip_Straight_1x10_Pitch2.54mm" H 5250 5750 60  0001 C CNN
 F 3 "" H 5250 5750 60  0001 C CNN
 	1    5250 5750
@@
 F 0 "U3" H 6750 5000 60  0000 C CNN
 F 1 "PRE-ADS1115" H 6550 6100 60  0000 C CNN
-F 2 "" H 6550 5750 60  0001 C CNN
+F 2 "Socket_Strips:Socket_Strip_Straight_1x10_Pitch2.54mm" H 6550 5750 60  0001 C CNN
 F 3 "" H 6550 5750 60  0001 C CNN
 	1    6550 5750
@@
 F 0 "U1" H 6800 8050 60  0000 C CNN
 F 1 "PRE-PCA9685" H 5300 8050 60  0000 C CNN
-F 2 "" H 5100 7550 60  0001 C CNN
+F 2 "FoxWestern:PCA9685" H 5100 7550 60  0001 C CNN
 F 3 "" H 5100 7550 60  0001 C CNN
 	1    5100 7550
@@
 F 0 "U9" H 11250 4950 60  0000 C CNN
 F 1 "PRE-ADS1115" H 11050 6050 60  0000 C CNN
-F 2 "" H 11050 5700 60  0001 C CNN
+F 2 "Socket_Strips:Socket_Strip_Straight_1x10_Pitch2.54mm" H 11050 5700 60  0001 C CNN
 F 3 "" H 11050 5700 60  0001 C CNN
 	1    11050 5700
@@
 F 0 "U5" H 9500 5050 60  0000 C CNN
 F 1 "PRE-ADS1115" H 9300 6150 60  0000 C CNN
-F 2 "" H 9300 5800 60  0001 C CNN
+F 2 "Socket_Strips:Socket_Strip_Straight_1x10_Pitch2.54mm" H 9300 5800 60  0001 C CNN
 F 3 "" H 9300 5800 60  0001 C CNN
 	1    9300 5800
@@
 F 0 "U4" H 11200 8050 60  0000 C CNN
 F 1 "PRE-PCA9685" H 9700 8050 60  0000 C CNN
-F 2 "" H 9500 7550 60  0001 C CNN
+F 2 "FoxWestern:PCA9685" H 9500 7550 60  0001 C CNN
 F 3 "" H 9500 7550 60  0001 C CNN
 	1    9500 7550
@@
 F 0 "R11" V 15180 1400 50  0000 C CNN
 F 1 "2.2K" V 15100 1400 50  0000 C CNN
-F 2 "" V 15030 1400 50  0001 C CNN
+F 2 "Resistors_SMD:R_0805" V 15030 1400 50  0001 C CNN
 F 3 "" H 15100 1400 50  0001 C CNN
 	1    15100 1400
@@
 F 0 "R12" V 15430 1400 50  0000 C CNN
 F 1 "2.2K" V 15350 1400 50  0000 C CNN
-F 2 "" V 15280 1400 50  0001 C CNN
+F 2 "Resistors_SMD:R_0805" V 15280 1400 50  0001 C CNN
 F 3 "" H 15350 1400 50  0001 C CNN
 	1    15350 1400
@@
 F 0 "R3" V 13430 1400 50  0000 C CNN
 F 1 "2.2K" V 13350 1400 50  0000 C CNN
-F 2 "" V 13280 1400 50  0001 C CNN
+F 2 "Resistors_SMD:R_0805" V 13280 1400 50  0001 C CNN
 F 3 "" H 13350 1400 50  0001 C CNN
 	1    13350 1400
@@
 F 0 "R4" V 13680 1400 50  0000 C CNN
 F 1 "2.2K" V 13600 1400 50  0000 C CNN
-F 2 "" V 13530 1400 50  0001 C CNN
+F 2 "Resistors_SMD:R_0805" V 13530 1400 50  0001 C CNN
 F 3 "" H 13600 1400 50  0001 C CNN
 	1    13600 1400
@@
 F 0 "R5" V 14280 1400 50  0000 C CNN
 F 1 "2.2K" V 14200 1400 50  0000 C CNN
-F 2 "" V 14130 1400 50  0001 C CNN
+F 2 "Resistors_SMD:R_0805" V 14130 1400 50  0001 C CNN
 F 3 "" H 14200 1400 50  0001 C CNN
 	1    14200 1400
@@
 F 0 "R10" V 14530 1400 50  0000 C CNN
 F 1 "2.2K" V 14450 1400 50  0000 C CNN
-F 2 "" V 14380 1400 50  0001 C CNN
+F 2 "Resistors_SMD:R_0805" V 14380 1400 50  0001 C CNN
 F 3 "" H 14450 1400 50  0001 C CNN
 	1    14450 1400
@@
 F 0 "J11" H 12100 2250 50  0000 C CNN
 F 1 "RFD900" V 12100 1800 50  0000 C CNN
-F 2 "Pin_Headers:Pin_Header_Straight_2x08_Pitch2.54mm" H 12100 600 50  0001 C CNN
+F 2 "Socket_Strips:Socket_Strip_Angled_2x08_Pitch2.54mm" H 12100 600 50  0001 C CNN
 F 3 "" H 12100 600 50  0001 C CNN
 	1    12100 1800
@@
 F 0 "U7" H 10250 3250 60  0000 C CNN
 F 1 "LM340MP-5.0" H 9850 3650 60  0000 C CNN
-F 2 "" H 9900 3350 60  0001 C CNN
+F 2 "TO_SOT_Packages_SMD:SOT-223-3Lead_TabPin2" H 9900 3350 60  0001 C CNN
 F 3 "" H 9900 3350 60  0001 C CNN
 	1    9900 3350
@@
 $EndComp
 $Comp
-L NucleoF411RE J5
-U 1 1 5939039A
-P 3400 2850
-F 0 "J5" H 3400 3850 50  0000 C CNN
-F 1 "NucleoF411RE" V 3400 2850 50  0000 C CNN
-F 2 "Pin_Headers:Pin_Header_Straight_2x19_Pitch2.54mm" H 3400 1850 50  0001 C CNN
-F 3 "" H 3400 1850 50  0001 C CNN
-	1    3400 2850
-	1    0    0    -1
-$EndComp
-$Comp
-L NucleoF411RE J5
-U 2 1 59390423
-P 5650 2850
-F 0 "J5" H 5650 3850 50  0000 C CNN
-F 1 "NucleoF411RE" V 5650 2850 50  0000 C CNN
-F 2 "Pin_Headers:Pin_Header_Straight_2x19_Pitch2.54mm" H 5650 1850 50  0001 C CNN
-F 3 "" H 5650 1850 50  0001 C CNN
-	2    5650 2850
-	1    0    0    -1
-$EndComp
-$Comp
 L +3V3 #PWR045
 U 1 1 59392483
@@
 F 0 "R13" V 14680 6150 50  0000 C CNN
 F 1 "220" V 14600 6150 50  0000 C CNN
-F 2 "" V 14530 6150 50  0001 C CNN
+F 2 "Resistors_SMD:R_0805" V 14530 6150 50  0001 C CNN
 F 3 "" H 14600 6150 50  0001 C CNN
 	1    14600 6150
@@
 F 0 "J20" H 13550 8650 50  0000 C CNN
 F 1 "GPS" V 13650 8150 50  0000 C CNN
-F 2 "Pin_Headers:Pin_Header_Straight_1x09_Pitch2.54mm" H 13550 8150 50  0001 C CNN
+F 2 "Socket_Strips:Socket_Strip_Straight_1x09_Pitch2.54mm" H 13550 8150 50  0001 C CNN
 F 3 "" H 13550 8150 50  0001 C CNN
 	1    13550 8150
@@
 F 0 "J21" H 15000 9250 50  0000 C CNN
 F 1 "COMPASS" V 15100 8900 50  0000 C CNN
-F 2 "Pin_Headers:Pin_Header_Straight_1x06_Pitch2.54mm" H 15000 8900 50  0001 C CNN
+F 2 "Socket_Strips:Socket_Strip_Straight_1x06_Pitch2.54mm" H 15000 8900 50  0001 C CNN
 F 3 "" H 15000 8900 50  0001 C CNN
 	1    15000 8900
@@
 F 0 "J14" H 14550 8150 50  0000 C CNN
 F 1 "ARDUINO NANO LEFT" V 14650 7350 50  0000 C CNN
-F 2 "Pin_Headers:Pin_Header_Straight_1x15_Pitch2.54mm" H 14550 7350 50  0001 C CNN
+F 2 "Socket_Strips:Socket_Strip_Straight_1x15_Pitch2.54mm" H 14550 7350 50  0001 C CNN
 F 3 "" H 14550 7350 50  0001 C CNN
 	1    14550 7350
@@
 F 0 "J22" H 14950 8150 50  0000 C CNN
 F 1 "ARDUINO NANO RIGHT" V 15050 7350 50  0000 C CNN
-F 2 "Pin_Headers:Pin_Header_Straight_1x15_Pitch2.54mm" H 14950 7350 50  0001 C CNN
+F 2 "Socket_Strips:Socket_Strip_Straight_1x15_Pitch2.54mm" H 14950 7350 50  0001 C CNN
 F 3 "" H 14950 7350 50  0001 C CNN
 	1    14950 7350
 	-1   0    0    -1
 $EndComp
+$Comp
+L CONN_02X19 J5
+U 1 1 593A19C2
+P 3400 2850
+F 0 "J5" H 3400 3850 50  0000 C CNN
+F 1 "NucleoLeft" V 3400 2850 50  0000 C CNN
+F 2 "Socket_Strips:Socket_Strip_Straight_2x19_Pitch2.54mm" H 3400 1850 50  0001 C CNN
+F 3 "" H 3400 1850 50  0001 C CNN
+	1    3400 2850
+	1    0    0    -1
+$EndComp
+$Comp
+L CONN_02X19 J23
+U 1 1 593A1A91
+P 5650 2850
+F 0 "J23" H 5650 3850 50  0000 C CNN
+F 1 "NucleoRight" V 5650 2850 50  0000 C CNN
+F 2 "Socket_Strips:Socket_Strip_Straight_2x19_Pitch2.54mm" H 5650 1850 50  0001 C CNN
+F 3 "" H 5650 1850 50  0001 C CNN
+	1    5650 2850
+	1    0    0    -1
+$EndComp
+$Comp
+L TL1963 U6
+U 1 1 593A6BB4
+P 9900 1650
+F 0 "U6" H 10250 1350 60  0000 C CNN
+F 1 "TL1963" H 9850 1850 60  0000 C CNN
+F 2 "TO_SOT_Packages_SMD:SOT-223-3Lead_TabPin2" H 9800 1700 60  0001 C CNN
+F 3 "" H 9800 1700 60  0001 C CNN
+	1    9900 1650
+	1    0    0    -1
+$EndComp
 $EndSCHEMATC
